Commit message: with kinect

File: common_sensors/urdf/sensors/kinect.urdf.xacro (robot description, xacro)
@@ -9,6 +9,8 @@
 	<xacro:macro name="sensor_kinect" params="parent">
 		<joint name="camera_rgb_joint" type="fixed">
-		      <origin xyz="${cam_px} ${cam_py} ${cam_pz}"
-			      rpy="${cam_or} ${cam_op} ${cam_oy}"/>
+		      <!--OJ <origin xyz="${cam_px} ${cam_py} ${cam_pz}"
+			      rpy="${cam_or} ${cam_op} ${cam_oy}"/> -->
+				  <origin xyz=" 0 0 1 "
+			      rpy= " 0 1.25 1.54 "/>
 			<parent link="${parent}"/>
 			<child link="camera_rgb_frame" />
@@ -34,5 +36,5 @@
 		</link>
 		<joint name="camera_joint" type="fixed">
-			<origin xyz="-0.031 ${-cam_py} -0.016" rpy="0 0 0"/>
+			<origin xyz="-0.031 ${-0} -0.016" rpy="0 0 0"/>
 			<parent link="camera_rgb_frame"/>
 			<child link="camera_link"/>
@@ -61,5 +63,5 @@
 		 (Hence, don't publish them additionally!) -->
 		<joint name="camera_depth_joint" type="fixed">
-			<origin xyz="0 ${2 * -cam_py} 0" rpy="0 0 0" />
+			<origin xyz="0 ${2 * -0} 0" rpy="0 0 0" />
 			<parent link="camera_rgb_frame" />
 			<child link="camera_depth_frame" />

File: common_sensors/urdf/sensors/kinect2_properties.urdf (Kopie).xacro (robot description, xacro)
@@ -4,12 +4,4 @@
        xmlns:interface="http://playerstage.sourceforge.net/gazebo/xmlschema/#interface"
        xmlns:xacro="http://www.ros.org/wiki/xacro">
-       <!-- OJ added this lines, see
-       https://roboticscasual.com/ros-tutorial-how-to-use-a-depth-camera-with-moveit-for-collision-avoidance/
-	<property name="cam_px" value="0.0" />
-	<property name="cam_py" value="0.0" />
-	<property name="cam_pz" value="1.0" />
-	<property name="cam_or" value="0" />
-	<property name="cam_op" value="1.25" />
-	<property name="cam_oy" value="1.54" /> -->
   <xacro:property name="VELOCITY_LIMIT_SCALE" value="0.6" />
   <!-- Gear Ratio Corrections: Divide transmission reductions by these factors (Nominally 1)-->

File: common_sensors/urdf/sensors/kinect_properties.urdf (Kopie).xacro (robot description, xacro)
@@ -12,9 +12,9 @@
 	<!-- OJ added this lines, see
        https://roboticscasual.com/ros-tutorial-how-to-use-a-depth-camera-with-moveit-for-collision-avoidance/  -->
-	<!--<property name="cam_px" value="0.0" />
+	<property name="cam_px" value="0.0" />
 	<property name="cam_py" value="0.0" />
 	<property name="cam_pz" value="1.0" />
 	<property name="cam_or" value="0" />
 	<property name="cam_op" value="1.25" />
-	<property name="cam_oy" value="1.54" /> -->
+	<property name="cam_oy" value="1.54" />
 </root>

Commit message: yep

File: common_sensors/urdf/sensors/kinect.urdf.xacro (robot description, xacro)
@@ -9,6 +9,10 @@
 	<xacro:macro name="sensor_kinect" params="parent">
 		<joint name="camera_rgb_joint" type="fixed">
-		      <!--OJ <origin xyz="${cam_px} ${cam_py} ${cam_pz}"
-			      rpy="${cam_or} ${cam_op} ${cam_oy}"/> -->
+		      <!--OJ cam_px cam_py not defined ?? Warum
+			  hier erstmal durch Zahlenwerte ersetzen, wir wollen nachher sowieso einen anderen Sensor nutzen
+			  <origin xyz="${cam_px} ${cam_py} ${cam_pz}"
+			      rpy="${cam_or} ${cam_op} ${cam_oy}"/>
+				  2 weiter cam_py weiter unten
+				  -->
 				  <origin xyz=" 0 0 1 "
 			      rpy= " 0 1.25 1.54 "/>

Commit message: cam_px problem solved

File: common_sensors/urdf/sensors/kinect.urdf.xacro (robot description, xacro)
@@ -2,19 +2,29 @@
 <root name="sensor_kinect" xmlns:xacro="http://ros.org/wiki/xacro">
 	<xacro:include filename="$(find common_sensors)/urdf/sensors/kinect_gazebo.xacro" />
-  <xacro:include filename="$(find common_sensors)/urdf/sensors/kinect_properties.urdf.xacro"/>
+  <!--OJ
+  not needed, properties are here
+  <xacro:include filename="$(find common_sensors)/urdf/sensors/kinect_properties.urdf.xacro"/> -->
   <!-- camera_name has to be unique! -->
   <xacro:kinect_sensor link_name="camera_depth_frame" camera_name="camera1"
                        frame_name="camera_depth_optical_frame"/>
 	<!-- Parameterised in part by the values in kinect_properties.urdf.xacro -->
-	<xacro:macro name="sensor_kinect" params="parent">
-		<joint name="camera_rgb_joint" type="fixed">
-		      <!--OJ cam_px cam_py not defined ?? Warum
+	<!--OJ cam_px cam_py not defined ?? Warum
 			  hier erstmal durch Zahlenwerte ersetzen, wir wollen nachher sowieso einen anderen Sensor nutzen
 			  <origin xyz="${cam_px} ${cam_py} ${cam_pz}"
 			      rpy="${cam_or} ${cam_op} ${cam_oy}"/>
 				  2 weiter cam_py weiter unten
-				  -->
 				  <origin xyz=" 0 0 1 "
-			      rpy= " 0 1.25 1.54 "/>
+			      rpy= " 0 1.25 1.54 "/> -->
+	<!-- mit xacro: davor hier einfügen funkt auch, wieos nicht per include-->
+	<xacro:property name="cam_px" value="0.0" />
+	<xacro:property name="cam_py" value="0.0" />
+	<xacro:property name="cam_pz" value="1.0" />
+	<xacro:property name="cam_or" value="0" />
+	<xacro:property name="cam_op" value="1.25" />
+	<xacro:property name="cam_oy" value="1.54" />
+	<xacro:macro name="sensor_kinect" params="parent">
+		<joint name="camera_rgb_joint" type="fixed">
+		    <origin xyz="${cam_px} ${cam_py} ${cam_pz}"
+			        rpy="${cam_or} ${cam_op} ${cam_oy}"/>
 			<parent link="${parent}"/>
 			<child link="camera_rgb_frame" />
@@ -40,5 +50,5 @@
 		</link>
 		<joint name="camera_joint" type="fixed">
-			<origin xyz="-0.031 ${-0} -0.016" rpy="0 0 0"/>
+			<origin xyz="-0.031 ${-cam_py} -0.016" rpy="0 0 0"/>
 			<parent link="camera_rgb_frame"/>
 			<child link="camera_link"/>
@@ -67,5 +77,5 @@
 		 (Hence, don't publish them additionally!) -->
 		<joint name="camera_depth_joint" type="fixed">
-			<origin xyz="0 ${2 * -0} 0" rpy="0 0 0" />
+			<origin xyz="0 ${2 * -cam_py} 0" rpy="0 0 0" />
 			<parent link="camera_rgb_frame" />
 			<child link="camera_depth_frame" />

File: common_sensors/urdf/sensors/kinect_properties.urdf.xacro (robot description, xacro)
@@ -1,5 +1,12 @@
 <?xml version="1.0"?>
 <root>
-  <!--
+	<xacro:property name="cam_px" value="0.0" />
+	<xacro:property name="cam_py" value="0.0" />
+	<xacro:property name="cam_pz" value="1.0" />
+	<xacro:property name="cam_or" value="0" />
+	<xacro:property name="cam_op" value="1.25" />
+	<xacro:property name="cam_oy" value="1.54" />
+</root>
+<!--
 	  Translation and rotation of camera from its base link
 	<property name="cam_px" value="0" />
@@ -12,9 +19,2 @@
 	<!-- OJ added this lines, see
        https://roboticscasual.com/ros-tutorial-how-to-use-a-depth-camera-with-moveit-for-collision-avoidance/  -->
-	<!--<property name="cam_px" value="0.0" />
-	<property name="cam_py" value="0.0" />
-	<property name="cam_pz" value="1.0" />
-	<property name="cam_or" value="0" />
-	<property name="cam_op" value="1.25" />
-	<property name="cam_oy" value="1.54" /> -->
-</root>
